File: DAUGHTER_ALLin.sch (KiCad schematic (older format))
At the start: 15 parts, among them IC1 SN6501-Q1, J1 Conn_02x08_Odd_Even, T1 760390012, U1 IZL10T1A-SOIC8

Commit message: multicb version
Parts:
- removed D1, D2: BAT54C_SOT23, Package_TO_SOT_SMD:SOT-23, symbol VDDTECH_SYMBOLS:BAT54C_SOT23
- removed IC1: SN6501-Q1, VDDTECH_FOOTPRINTS:SOT95P280X145-5N, symbol VDDTECH_SYMBOLS:SN6501-Q1
- added C10, C7, C8, C9: C_0805_1u, Capacitor_SMD:C_0805_2012Metric_Pad1.15x1.40mm_HandSolder, symbol VDDTECH_SYMBOLS:C_0805_1u
- added C11, C6: C_0805, Capacitor_SMD:C_0805_2012Metric_Pad1.15x1.40mm_HandSolder, symbol VDDTECH_SYMBOLS:C_0805
- added D1, D2: MBR0520, Diode_SMD:D_SOD-123, symbol Diode:MBR0520
- added IC1: ADUM3190BRQZ, VDDTECH_FOOTPRINTS:SOP64P600X175-16N, symbol VDDTECH_SYMBOLS:ADUM3190BRQZ
- added JP1: SolderJumper_2_Open_VDDTECH, Jumper:SolderJumper-2_P1.3mm_Open_RoundedPad1.0x1.5mm, symbol VDDTECH_SYMBOLS:SolderJumper_2_Open_VDDTECH
- added R3: Heater, Resistor_SMD:R_2010_5025Metric_Pad1.52x2.65mm_HandSolder, symbol Device:Heater
- added R4, R7, R8: 10k R_0603, Resistor_SMD:R_0603_1608Metric, symbol VDDTECH_SYMBOLS:R_0603
- added R9: R_0603, Resistor_SMD:R_0603_1608Metric_Pad1.05x0.95mm_HandSolder, symbol VDDTECH_SYMBOLS:R_0603
- added U2: SN6505BDBV, Package_TO_SOT_SMD:SOT-23-6, symbol Power_Management:SN6505BDBV
- added U3: TPS76350, Package_TO_SOT_SMD:SOT-23-5, symbol Regulator_Linear:TPS76350
- U1: footprint VDDTECH_FOOTPRINTS:SOIC8_typ_HEAT -> VDDTECH_FOOTPRINTS:SOIC8_typ_HEAT_no_vias
Connections:
- net labels added: EAOUT, EAOUT2, REFOUT1, REFOUT2, VDD_heat, VREG1, VREG2
- net labels removed: R_HEAT_SW
- wire segments 55 -> 97
Other:
- note removed: "High side isolator"
- moved on the sheet: C1, C2, C3, R6, U1
